Commit message: Editting module carts import

File: azenta_description/urdf/peeler_robot.xacro (robot description, xacro)
@@ -1,13 +1,18 @@
 <?xml version="1.0"?>
 <robot name="Peeler_Robot" xmlns:xacro="http://www.ros.org/wiki/xacro">
-  <!-- Materials -->
-  <material name="white">
-    <color rgba="1 1 1 1"/>
-  </material>
-  <material name="aluminum">
-    <color rgba="0.6 0.6 0.6 1"/>
-  </material>
+ <!-- Materials -->
+  <xacro:include filename="$(find azenta_description)/urdf/materials.xacro" />
+  <!-- Module Carts -->
+  <xacro:include filename="$(find azenta_description)/urdf/module_carts.urdf.xacro" />
+  <xacro:Module_Carts prefix="module_carts/"/>
   <!-- Peeler -->
   <xacro:include filename="$(find azenta_description)/urdf/peeler.urdf.xacro" />
   <xacro:Peeler prefix="peeler/"/>
+  <joint name="Peeler_Base" type="fixed">
+    <parent link="module_carts/cart_6"/>
+    <child link="peeler/peeler_base"/>
+    <axis xyz="0 0 0"/>
+    <origin xyz="-0.13 0.15 1.042" rpy="0 0 0"/>
+    <limit effort="1000.0" lower="0" upper="0" velocity="0.5"/>
+  </joint>
 </robot>

File: azenta_description/urdf/sealer_robot.xacro (robot description, xacro)
@@ -2,12 +2,17 @@
 <robot name="Sealer_Robot" xmlns:xacro="http://www.ros.org/wiki/xacro">
   <!-- Materials -->
-  <material name="white">
-    <color rgba="1 1 1 1"/>
-  </material>
-  <material name="aluminum">
-    <color rgba="0.6 0.6 0.6 1"/>
-  </material>
+  <xacro:include filename="$(find azenta_description)/urdf/materials.xacro" />
+  <!-- Module Carts -->
+  <xacro:include filename="$(find azenta_description)/urdf/module_carts.urdf.xacro" />
+  <xacro:Module_Carts prefix="module_carts/"/>
   <!-- Sealer -->
   <xacro:include filename="$(find azenta_description)/urdf/sealer.urdf.xacro" />
   <xacro:Sealer prefix="sealer/"/>
+  <joint name="Sealer_Base" type="fixed">
+    <parent link="module_carts/cart_6"/>
+    <child link="sealer/sealer_base"/>
+    <axis xyz="0 0 0"/>
+    <origin xyz="0.27 -0.53 1.042" rpy="0 0 0"/>
+    <limit effort="1000.0" lower="0" upper="0" velocity="0.5"/>
+  </joint>
 </robot>
