Commit message: Clean up

File: azenta_description/urdf/peeler.urdf.xacro (robot description, xacro)
@@ -7,5 +7,5 @@
       <origin xyz="0 0 0" rpy="1.5708 0 0"/>
       <geometry>
-        <mesh filename="package://pf400_description/meshes/peeler_base.STL" scale="0.001 0.001 0.001"/>
+        <mesh filename="package://azenta_description/meshes/peeler_base.STL" scale="0.001 0.001 0.001"/>
       </geometry>
       <material name="light_blue"/>
@@ -13,5 +13,5 @@
     <collision>
       <geometry>
-        <mesh filename="package://pf400_description/meshes/peeler_base.STL" scale="0.001 0.001 0.001"/>
+        <mesh filename="package://azenta_description/meshes/peeler_base.STL" scale="0.001 0.001 0.001"/>
       </geometry>
       <origin xyz="0 0 0" rpy="1.5708 0 0"/>
@@ -22,5 +22,5 @@
       <origin xyz="0 0 0" rpy="0 1.5708 0"/>
       <geometry>
-        <mesh filename="package://pf400_description/meshes/peeler_plate.STL" scale="0.001 0.001 0.001"/>
+        <mesh filename="package://azenta_description/meshes/peeler_plate.STL" scale="0.001 0.001 0.001"/>
       </geometry>
       <material name="white"/>
@@ -28,5 +28,5 @@
     <collision>
       <geometry>
-        <mesh filename="package://pf400_description/meshes/peeler_plate.STL" scale="0.001 0.001 0.001"/>
+        <mesh filename="package://azenta_description/meshes/peeler_plate.STL" scale="0.001 0.001 0.001"/>
       </geometry>
       <origin xyz="0 0 0" rpy="0 1.5708 0"/>
@@ -34,5 +34,5 @@
   </link>
   <!-- Joints -->
-  <joint name="Peeler_Plate_Joint" type="fixed">
+  <joint name="Peeler_Plate_Joint" type="revolute">
     <parent link="${prefix}peeler_base"/>
     <child link="${prefix}peeler_plate"/>

File: azenta_description/urdf/sealer.urdf.xacro (robot description, xacro)
@@ -7,5 +7,5 @@
       <origin xyz="0 0 0" rpy="1.5708 0 1.5708"/>
       <geometry>
-        <mesh filename="package://pf400_description/meshes/sealer_base.STL" scale="0.001 0.001 0.001"/>
+        <mesh filename="package://azenta_description/meshes/sealer_base.STL" scale="0.001 0.001 0.001"/>
       </geometry>
       <material name="pink"/>
@@ -13,5 +13,5 @@
     <collision>
       <geometry>
-        <mesh filename="package://pf400_description/meshes/sealer_base.STL" scale="0.001 0.001 0.001"/>
+        <mesh filename="package://azenta_description/meshes/sealer_base.STL" scale="0.001 0.001 0.001"/>
       </geometry>
       <origin xyz="0 0 0" rpy="1.5708 0 1.5708"/>
@@ -22,5 +22,5 @@
       <origin xyz="0 0 0" rpy="0 1.5708 0"/>
       <geometry>
-        <mesh filename="package://pf400_description/meshes/sealer_plate.STL" scale="0.001 0.001 0.001"/>
+        <mesh filename="package://azenta_description/meshes/sealer_plate.STL" scale="0.001 0.001 0.001"/>
       </geometry>
       <material name="aluminum"/>
@@ -28,5 +28,5 @@
     <collision>
       <geometry>
-        <mesh filename="package://pf400_description/meshes/sealer_plate.STL" scale="0.001 0.001 0.001"/>
+        <mesh filename="package://azenta_description/meshes/sealer_plate.STL" scale="0.001 0.001 0.001"/>
       </geometry>
       <origin xyz="0 0 0" rpy="0 1.5708 0"/>
@@ -34,5 +34,5 @@
   </link>
   <!-- Joints -->
-  <joint name="Sealer_Plate_Joint" type="fixed">
+  <joint name="Sealer_Plate_Joint" type="revolute">
     <parent link="${prefix}sealer_base"/>
     <child link="${prefix}sealer_plate"/>

Commit message: Changing joint type

File: azenta_description/urdf/peeler.urdf.xacro (robot description, xacro)
@@ -34,5 +34,5 @@
   </link>
   <!-- Joints -->
-  <joint name="Peeler_Plate_Joint" type="revolute">
+  <joint name="Peeler_Plate_Joint" type="prismatic">
     <parent link="${prefix}peeler_base"/>
     <child link="${prefix}peeler_plate"/>

File: azenta_description/urdf/sealer.urdf.xacro (robot description, xacro)
@@ -34,5 +34,5 @@
   </link>
   <!-- Joints -->
-  <joint name="Sealer_Plate_Joint" type="revolute">
+  <joint name="Sealer_Plate_Joint" type="prismatic">
     <parent link="${prefix}sealer_base"/>
     <child link="${prefix}sealer_plate"/>

Commit message: Clean up

File: azenta_description/urdf/peeler.urdf.xacro (robot description, xacro)
@@ -39,5 +39,5 @@
     <axis xyz="0 0 1"/>
     <origin xyz="0.25 -0.18 0.083" rpy="1.5708 0 0"/>
-    <limit effort="1000.0" lower="0" upper="0.3" velocity="0.5"/>
+    <limit effort="1000.0" lower="0.0" upper="0.3" velocity="0.5"/>
   </joint>
   </xacro:macro>

File: azenta_description/urdf/sealer.urdf.xacro (robot description, xacro)
@@ -39,5 +39,5 @@
     <axis xyz="0 0 1"/>
     <origin xyz="0.057 0.28 0.01" rpy="1.5708 0 0"/>
-    <limit effort="1000.0" lower="0" upper="0.25" velocity="0.5"/>
+    <limit effort="1000.0" lower="0.0" upper="0.25" velocity="0.5"/>
   </joint>
   </xacro:macro>

Commit message: Update

File: azenta_description/urdf/peeler.urdf.xacro (robot description, xacro)
@@ -3,5 +3,5 @@
   <!-- Links -->
   <xacro:macro name="Peeler" params = "prefix">
-    <link name="${prefix}peeler_base">
+  <link name="${prefix}peeler_base">
     <visual>
       <origin xyz="0 0 0" rpy="1.5708 0 0"/>
